Commit message: simplified ceres_urdf file structure

File: src/ceres_urdf/urdf/ceres.xacro (robot description, xacro)
@@ -13,5 +13,5 @@
         <visual>
             <geometry>
-                <mesh filename="package://ceres_urdf/meshes/cycloidal_drive/base_struct.stl" scale="0.001 0.001 0.001"/>
+                <box size="0.30670 0.1600 0.135"/>
             </geometry>
             <origin xyz="0 0 0" rpy="1.57 0 0" />
@@ -20,7 +20,6 @@
         <collision>
             <geometry>
-                <mesh filename="package://ceres_urdf/meshes/cycloidal_drive/base_struct.stl" scale="0.001 0.001 0.001"/>
+                <box size="0.30670 0.1600 0.135"/>
             </geometry>
-            <origin xyz="0 0 0" rpy="1.57 0 0" />
             <material name="blue"/>
         </collision>
@@ -29,31 +28,14 @@
         <visual>
             <geometry>
-                <mesh filename="package://ceres_urdf/meshes/cycloidal_drive/base_pivot.stl" scale="0.001 0.001 0.001"/>
+                <box size="0.1633 0.1633 0.1633"/>
             </geometry>
-            <origin xyz="0.04887 0.05876 -0.06" rpy="1.34 -0.32 -1.389"/>
+            <origin xyz="0 0 0" rpy="0 0 0"/>
             <material name="red"/>
         </visual>
         <collision>
             <geometry>
-                <mesh filename="package://ceres_urdf/meshes/cycloidal_drive/base_pivot.stl" scale="0.001 0.001 0.001"/>
+                <box size="0.1633 0.1633 0.1633"/>
             </geometry>
-            <origin xyz="0.04887 0.05876 -0.06" rpy="1.34 -0.32 -1.389"/>
             <material name="red"/>
-        </collision>
-    </link>
-    <link name="shoulder_gearbox_link">
-        <visual>
-            <geometry>
-                <mesh filename="package://ceres_urdf/meshes/cycloidal_drive/shoulder_gearbox.stl" scale="0.001 0.001 0.001"/>
-            </geometry>
-            <origin xyz="0.105 -0.071 0.0715" rpy="0 1.57 1.57"/>
-            <material name="grey"/>
-        </visual>
-        <collision>
-            <geometry>
-                <mesh filename="package://ceres_urdf/meshes/cycloidal_drive/shoulder_gearbox.stl" scale="0.001 0.001 0.001"/>
-            </geometry>
-            <origin xyz="0.105 -0.071 0.0715" rpy="0 1.57 1.57"/>
-            <material name="grey"/>
         </collision>
     </link>
@@ -61,14 +43,13 @@
         <visual>
             <geometry>
-                <mesh filename="package://ceres_urdf/meshes/cycloidal_drive/bicep_tube.stl" scale="0.001 0.001 0.001"/>
+                <cylinder radius="0.0348" length="0.520"/>
             </geometry>
-            <origin xyz="0.1025 -0.192 -0.086" rpy="0 -0.15 1.57"/>
+            <origin xyz="0 0 0.220" rpy="0 0 0"/>
             <material name="grey"/>
         </visual>
         <collision>
             <geometry>
-                <mesh filename="package://ceres_urdf/meshes/cycloidal_drive/bicep_tube.stl" scale="0.001 0.001 0.001"/>
+                <cylinder radius="0.0348" length="0.520"/>
             </geometry>
-            <origin xyz="0.1025 -0.192 -0.086" rpy="0 -0.15 1.57"/>
             <material name="grey"/>
         </collision>
@@ -77,30 +58,43 @@
         <visual>
             <geometry>
-                <mesh filename="package://ceres_urdf/meshes/cycloidal_drive/bicep_gearbox.stl" scale="0.001 0.001 0.001"/>
+                <box size="0.11615 0.158 0.170"/>
             </geometry>
-            <origin xyz="0.0190 -0.099 -0.092" rpy="0 -0.15 1.57"/>
+            <origin xyz="0 0 0" rpy="0 0 0"/>
             <material name="red"/>
         </visual>
         <collision>
             <geometry>
-                <mesh filename="package://ceres_urdf/meshes/cycloidal_drive/bicep_gearbox.stl" scale="0.001 0.001 0.001"/>
+                <box size="0.11615 0.158 0.170"/>
             </geometry>
-            <origin xyz="0.0190 -0.099 -0.092" rpy="0 -0.15 1.57"/>
             <material name="red"/>
         </collision>
     </link>
-    <link name="forearm_tube_link">
+   <link name="forearm_tube_link">
         <visual>
             <geometry>
-                <mesh filename="package://ceres_urdf/meshes/cycloidal_drive/forearm_tube.stl" scale="0.001 0.001 0.001"/>
+                <cylinder radius="0.03810" length="0.300"/>
             </geometry>
-            <origin xyz="0.02678 -0.0094 -0.54" rpy="0 0 2.09"/>
+            <origin xyz="0 0 0.150" rpy="0 0 0"/>
             <material name="grey"/>
         </visual>
         <collision>
             <geometry>
-                <mesh filename="package://ceres_urdf/meshes/cycloidal_drive/forearm_tube.stl" scale="0.001 0.001 0.001"/>
+                <cylinder radius="0.03810" length="0.300"/>
             </geometry>
-            <origin xyz="0.02678 -0.0094 -0.54" rpy="0 0 2.09"/>
+            <material name="grey"/>
+        </collision>
+    </link>
+     <link name="bracket_connection_link">
+        <visual>
+            <geometry>
+                <box size="0.008 0.10030 0.14015"/>
+            </geometry>
+            <origin xyz="0 0 0" rpy="0 0 0"/>
+            <material name="grey"/>
+        </visual>
+        <collision>
+            <geometry>
+                <box size="0 0 0"/>
+            </geometry>
             <material name="grey"/>
         </collision>
@@ -109,30 +103,13 @@
         <visual>
             <geometry>
-                <mesh filename="package://ceres_urdf/meshes/cycloidal_drive/wrist_gearbox.stl" scale="0.001 0.001 0.001"/>
+                <box size="0.04445 0.06200 0.07"/>
             </geometry>
-            <origin xyz="-0.05 0.055 0.040" rpy="0 1.38 -1.57"/>
-            <material name="red"/>
-        </visual>
-        <collision>
-            <geometry>
-                <mesh filename="package://ceres_urdf/meshes/cycloidal_drive/wrist_gearbox.stl" scale="0.001 0.001 0.001"/>
-            </geometry>
-            <origin xyz="-0.05 0.055 0.040" rpy="0 1.38 -1.57"/>
-            <material name="red"/>
-        </collision>
-    </link>
-    <link name="gripper_gearbox_link">
-        <visual>
-            <geometry>
-                <mesh filename="package://ceres_urdf/meshes/cycloidal_drive/gripper_gearbox.stl" scale="0.001 0.001 0.001"/>
-            </geometry>
-            <origin xyz="0.011 -0.205 0.020" rpy="0 1.57 1.57"/>
+            <origin xyz="0 0 0" rpy="0 0 0"/>
             <material name="grey"/>
         </visual>
         <collision>
             <geometry>
-                <mesh filename="package://ceres_urdf/meshes/cycloidal_drive/gripper_gearbox.stl" scale="0.001 0.001 0.001"/>
+                <box size="0 0 0"/>
             </geometry>
-            <origin xyz="0.011 -0.205 0.020" rpy="0 1.57 1.57"/>
             <material name="grey"/>
         </collision>
@@ -141,14 +118,13 @@
         <visual>
             <geometry>
-                <mesh filename="package://ceres_urdf/meshes/cycloidal_drive/gripper_claw.stl" scale="0.001 0.001 0.001"/>
+                <box size="0.033 0.14759 0.24761"/>
             </geometry>
-            <origin xyz="0.016 -0.246 0.0736" rpy="-1.57 1.57 0"/>
+            <origin xyz="0 0 0" rpy="0 0 0"/>
             <material name="blue"/>
         </visual>
         <collision>
             <geometry>
-                <mesh filename="package://ceres_urdf/meshes/cycloidal_drive/gripper_claw.stl" scale="0.001 0.001 0.001"/>
+                <box size="0.033 0.14759 0.24761"/>
             </geometry>
-            <origin xyz="0.016 -0.246 0.0736" rpy="-1.57 1.57 0"/>
             <material name="blue"/>
         </collision>
@@ -157,46 +133,40 @@
         <parent link="base_structure_link"/>
         <child link="base_pivot_link"/>
-        <origin xyz="0.156 -0.074 0.104" rpy="0 0 0"/>
+        <origin xyz="0 0 0.1618" rpy="0 0 0"/>
         <axis xyz="0 0 1"/>
     </joint>
-    <joint name="base_pivot_shoulder_gearbox_joint" type="continuous">
+    <joint name="base_bicep_tube_joint" type="continuous">
         <parent link="base_pivot_link"/>
-        <child link="shoulder_gearbox_link"/>
-        <origin xyz="0 0 0.082" rpy="0 0 0"/>
+        <child link="bicep_tube_link"/>
+        <origin xyz="0.11645 0 0" rpy="0 0 0"/>
+    </joint>
+    <joint name="bicep_gearbox_joint" type="continuous">
+        <parent link="bicep_tube_link"/>
+        <child link="bicep_gearbox_link"/>
+        <origin xyz="-0.092875 0 0.440" rpy="0 0 0"/>
         <axis xyz="1 0 0"/>
     </joint>
-    <joint name="shoulder_tube_joint" type="fixed">
-        <parent link="shoulder_gearbox_link"/>
-        <child link="bicep_tube_link"/>
-        <origin xyz="0 0 0" rpy="0 0 0"/>
-    </joint>
-    <joint name="bicep_tube_gearbox_joint" type="continuous">
-        <parent link="bicep_tube_link"/>
-        <child link="bicep_gearbox_link"/>
-        <origin xyz="0.0837 -0.224 0.3530" rpy="0 0 0"/>
-        <axis xyz="1 0 0"/>
-    </joint>
-    <joint name="bicep_gearbox_forearm_tube_joint" type="fixed">
+   <joint name="gearbox_forearm_joint" type="fixed">
         <parent link="bicep_gearbox_link"/>
         <child link="forearm_tube_link"/>
-        <origin xyz="-0.09562 -0.058 0.01" rpy="2.181 0 0"/>
+        <origin xyz="0 0 0.085" rpy="0 0 0"/>
         <axis xyz=" 0 0 1"/>
     </joint>
-    <joint name="forearm_tube_wrist_gearbox_joint" type="continuous">
+    <joint name="forearm_bracket_joint" type="continuous">
         <parent link="forearm_tube_link"/>
-        <child link="wrist_gearbox_link"/>
-        <origin xyz="0 0 0.345" rpy="0 0 0"/>
+        <child link="bracket_connection_link"/>
+        <origin xyz="0.0421 0 0.3" rpy="0 0 0"/>
         <axis xyz=" 1 0 0"/>
     </joint>
-    <joint name="wrist_gearbox_gripper_gearbox_joint" type="fixed">
+    <joint name="bracket_wrist_joint" type="fixed">
+        <parent link="bracket_connection_link"/>
+        <child link="wrist_gearbox_link"/>
+        <origin xyz="-0.026225 0 0.070075" rpy="0 0 0"/>
+    </joint>
+    <joint name="wrist_gripper_joint" type="continuous">
         <parent link="wrist_gearbox_link"/>
-        <child link="gripper_gearbox_link"/>
-        <origin xyz="0 0 0" rpy="0 0 0"/>
-    </joint>
-     <joint name="gripper_claw_joint" type="continuous">
-        <parent link="gripper_gearbox_link"/>
         <child link="gripper_claw_link"/>
-        <origin xyz="-0.007 -0.11 -0.002" rpy="0 0 0"/>
-        <axis xyz="0 1 0"/>
+        <origin xyz="0.005725 0 0.159" rpy="0 0 0"/>
+        <axis xyz="0 0 1"/>
     </joint>
 </robot>

Commit message: modified ik files now fully functioning on Rviz

File: src/ceres_urdf/urdf/ceres.xacro (robot description, xacro)
@@ -130,22 +130,25 @@
         </collision>
     </link>
-    <joint name="base_structure_joint" type="continuous">
+    <joint name="joint1" type="continuous">
         <parent link="base_structure_link"/>
         <child link="base_pivot_link"/>
         <origin xyz="0 0 0.1618" rpy="0 0 0"/>
+        <limit effort="20" velocity="1.0" lower="-2.355" upper="1.57"/>
         <axis xyz="0 0 1"/>
     </joint>
-    <joint name="base_bicep_tube_joint" type="continuous">
+    <joint name="joint2" type="continuous">
         <parent link="base_pivot_link"/>
         <child link="bicep_tube_link"/>
         <origin xyz="0.11645 0 0" rpy="0 0 0"/>
+        <limit effort="20" velocity="1.0" lower="-0.785" upper="1.0467"/>
     </joint>
-    <joint name="bicep_gearbox_joint" type="continuous">
+    <joint name="joint3" type="continuous">
         <parent link="bicep_tube_link"/>
         <child link="bicep_gearbox_link"/>
         <origin xyz="-0.092875 0 0.440" rpy="0 0 0"/>
+        <limit effort="20" velocity="1.0" lower="-0.466" upper="1.989"/>
         <axis xyz="1 0 0"/>
     </joint>
-   <joint name="gearbox_forearm_joint" type="fixed">
+   <joint name="joint4" type="fixed">
         <parent link="bicep_gearbox_link"/>
         <child link="forearm_tube_link"/>
@@ -153,19 +156,21 @@
         <axis xyz=" 0 0 1"/>
     </joint>
-    <joint name="forearm_bracket_joint" type="continuous">
+    <joint name="joint5" type="continuous">
         <parent link="forearm_tube_link"/>
         <child link="bracket_connection_link"/>
         <origin xyz="0.0421 0 0.3" rpy="0 0 0"/>
+        <limit effort="20" velocity="1.0" lower="-1.57" upper="1.57"/>
         <axis xyz=" 1 0 0"/>
     </joint>
-    <joint name="bracket_wrist_joint" type="fixed">
+    <joint name="joint6" type="fixed">
         <parent link="bracket_connection_link"/>
         <child link="wrist_gearbox_link"/>
         <origin xyz="-0.026225 0 0.070075" rpy="0 0 0"/>
     </joint>
-    <joint name="wrist_gripper_joint" type="continuous">
+    <joint name="joint7" type="continuous">
         <parent link="wrist_gearbox_link"/>
         <child link="gripper_claw_link"/>
         <origin xyz="0.005725 0 0.159" rpy="0 0 0"/>
+        <limit effort="20" velocity="1.0" lower="-3.14" upper="3.14"/>
         <axis xyz="0 0 1"/>
     </joint>

Commit message: added joint limits for arm

File: src/ceres_urdf/urdf/ceres.xacro (robot description, xacro)
@@ -1,3 +1,3 @@
-<?xml version="1.0"?>
+<?xml version="2.0"?>
 <robot name="ceres_rover" xmlns:xacro="http://www.ros.org/wiki/xacro">
     <material name="blue" >
@@ -134,5 +134,5 @@
         <child link="base_pivot_link"/>
         <origin xyz="0 0 0.1618" rpy="0 0 0"/>
-        <limit effort="20" velocity="1.0" lower="-2.355" upper="1.57"/>
+        <limit effort="20" velocity="2.0" lower="-2.355" upper="1.57"/>
         <axis xyz="0 0 1"/>
     </joint>
@@ -141,5 +141,5 @@
         <child link="bicep_tube_link"/>
         <origin xyz="0.11645 0 0" rpy="0 0 0"/>
-        <limit effort="20" velocity="1.0" lower="-0.785" upper="1.0467"/>
+        <limit effort="20" velocity="2.0" lower="-0.785" upper="2.0467"/>
     </joint>
     <joint name="joint3" type="continuous">
@@ -147,5 +147,5 @@
         <child link="bicep_gearbox_link"/>
         <origin xyz="-0.092875 0 0.440" rpy="0 0 0"/>
-        <limit effort="20" velocity="1.0" lower="-0.466" upper="1.989"/>
+        <limit effort="20" velocity="2.0" lower="-0.466" upper="1.989"/>
         <axis xyz="1 0 0"/>
     </joint>
@@ -156,9 +156,9 @@
         <axis xyz=" 0 0 1"/>
     </joint>
-    <joint name="joint5" type="continuous">
+    <joint name="joint5" type="revolute">
         <parent link="forearm_tube_link"/>
         <child link="bracket_connection_link"/>
         <origin xyz="0.0421 0 0.3" rpy="0 0 0"/>
-        <limit effort="20" velocity="1.0" lower="-1.57" upper="1.57"/>
+        <limit effort="20" velocity="2.0" lower="-1.57" upper="1.57"/>
         <axis xyz=" 1 0 0"/>
     </joint>
@@ -168,9 +168,9 @@
         <origin xyz="-0.026225 0 0.070075" rpy="0 0 0"/>
     </joint>
-    <joint name="joint7" type="continuous">
+    <joint name="joint7" type="revolute">
         <parent link="wrist_gearbox_link"/>
         <child link="gripper_claw_link"/>
         <origin xyz="0.005725 0 0.159" rpy="0 0 0"/>
-        <limit effort="20" velocity="1.0" lower="-3.14" upper="3.14"/>
+        <limit effort="20" velocity="2.0" lower="-3.14" upper="3.14"/>
         <axis xyz="0 0 1"/>
     </joint>

Commit message: added right and left claw (2 new links and 2 joints)

File: src/ceres_urdf/urdf/ceres.xacro (robot description, xacro)
@@ -118,14 +118,44 @@
         <visual>
             <geometry>
-                <box size="0.033 0.14759 0.24761"/>
-            </geometry>
-            <origin xyz="0 0 0" rpy="0 0 0"/>
-            <material name="blue"/>
-        </visual>
-        <collision>
-            <geometry>
-                <box size="0.033 0.14759 0.24761"/>
-            </geometry>
-            <material name="blue"/>
+                <box size="0.033 0.14759 0.070"/>
+            </geometry>
+            <origin xyz="0 0 0" rpy="0 0 0"/>
+            <material name="blue"/>
+        </visual>
+        <collision>
+            <geometry>
+                <box size="0.033 0.14759 0.070"/>
+            </geometry>
+            <material name="blue"/>
+        </collision>
+    </link>
+    <link name="right_claw_link">
+        <visual>
+            <geometry>
+                <box size="0.033 0.073795 0.200"/>
+            </geometry>
+            <origin xyz="0 0 0" rpy="0 0 0"/>
+            <material name="red"/>
+        </visual>
+        <collision>
+            <geometry>
+                <box size="0.033 0.073795 0.200"/>
+            </geometry>
+            <material name="red"/>
+        </collision>
+    </link>
+    <link name="left_claw_link">
+        <visual>
+            <geometry>
+                <box size="0.033 0.073795 0.200"/>
+            </geometry>
+            <origin xyz="0 0 0" rpy="0 0 0"/>
+            <material name="red"/>
+        </visual>
+        <collision>
+            <geometry>
+                <box size="0.033 0.073795 0.200"/>
+            </geometry>
+            <material name="red"/>
         </collision>
     </link>
@@ -171,7 +201,21 @@
         <parent link="wrist_gearbox_link"/>
         <child link="gripper_claw_link"/>
-        <origin xyz="0.005725 0 0.159" rpy="0 0 0"/>
+        <origin xyz="0.005725 0 0.07" rpy="0 0 0"/>
         <limit effort="20" velocity="2.0" lower="-3.14" upper="3.14"/>
         <axis xyz="0 0 1"/>
     </joint>
+    <joint name="joint8" type="prismatic">
+        <parent link="gripper_claw_link"/>
+        <child link="right_claw_link"/>
+        <origin xyz="0 0.036895 0.135" rpy="0 0 0"/>
+        <limit effort="20" velocity="2.0" lower="0" upper="0.05"/>
+        <axis xyz="0 1 0"/>
+    </joint>
+    <joint name="joint9" type="prismatic">
+        <parent link="gripper_claw_link"/>
+        <child link="left_claw_link"/>
+        <origin xyz="0 -0.036895 0.135" rpy="0 0 0"/>
+        <limit effort="20" velocity="2.0" lower="-0.05" upper="0"/>
+        <axis xyz="0 1 0"/>
+    </joint>
 </robot>

Commit message: updated claw limit

File: src/ceres_urdf/urdf/ceres.xacro (robot description, xacro)
@@ -209,5 +209,5 @@
         <child link="right_claw_link"/>
         <origin xyz="0 0.036895 0.135" rpy="0 0 0"/>
-        <limit effort="20" velocity="2.0" lower="0" upper="0.05"/>
+        <limit effort="20" velocity="2.0" lower="0" upper="0.0275"/>
         <axis xyz="0 1 0"/>
     </joint>
@@ -216,5 +216,5 @@
         <child link="left_claw_link"/>
         <origin xyz="0 -0.036895 0.135" rpy="0 0 0"/>
-        <limit effort="20" velocity="2.0" lower="-0.05" upper="0"/>
+        <limit effort="20" velocity="2.0" lower="-0.0275" upper="0"/>
         <axis xyz="0 1 0"/>
     </joint>

Commit message: modified

File: src/ceres_urdf/urdf/ceres.xacro (robot description, xacro)
@@ -1,3 +1,3 @@
-<?xml version="1.0"?>
+<?xml version="2.0"?>
 <robot name="ceres_rover" xmlns:xacro="http://www.ros.org/wiki/xacro">
     <material name="blue" >
@@ -164,5 +164,5 @@
         <child link="base_pivot_link"/>
         <origin xyz="0 0 0.1618" rpy="0 0 0"/>
-        <limit effort="20" velocity="2.0" lower="-2.355" upper="1.57"/>
+        <!-- <limit effort="20" velocity="2.0" lower="-2.355" upper="1.57"/> -->
         <axis xyz="0 0 1"/>
     </joint>
@@ -171,5 +171,5 @@
         <child link="bicep_tube_link"/>
         <origin xyz="0.11645 0 0" rpy="0 0 0"/>
-        <limit effort="20" velocity="2.0" lower="-0.785" upper="2.0467"/>
+        <!-- <limit effort="20" velocity="2.0" lower="-0.785" upper="2.0467"/> -->
     </joint>
     <joint name="joint3" type="continuous">
@@ -177,5 +177,5 @@
         <child link="bicep_gearbox_link"/>
         <origin xyz="-0.092875 0 0.440" rpy="0 0 0"/>
-        <limit effort="20" velocity="2.0" lower="-0.466" upper="1.989"/>
+        <!-- <limit effort="20" velocity="2.0" lower="-0.466" upper="1.989"/> -->
         <axis xyz="1 0 0"/>
     </joint>

Commit message: modified

File: src/ceres_urdf/urdf/ceres.xacro (robot description, xacro)
@@ -164,5 +164,4 @@
         <child link="base_pivot_link"/>
         <origin xyz="0 0 0.1618" rpy="0 0 0"/>
-        <!-- <limit effort="20" velocity="2.0" lower="-2.355" upper="1.57"/> -->
         <axis xyz="0 0 1"/>
     </joint>
@@ -171,5 +170,4 @@
         <child link="bicep_tube_link"/>
         <origin xyz="0.11645 0 0" rpy="0 0 0"/>
-        <!-- <limit effort="20" velocity="2.0" lower="-0.785" upper="2.0467"/> -->
     </joint>
     <joint name="joint3" type="continuous">
@@ -177,5 +175,4 @@
         <child link="bicep_gearbox_link"/>
         <origin xyz="-0.092875 0 0.440" rpy="0 0 0"/>
-        <!-- <limit effort="20" velocity="2.0" lower="-0.466" upper="1.989"/> -->
         <axis xyz="1 0 0"/>
     </joint>
@@ -190,5 +187,4 @@
         <child link="bracket_connection_link"/>
         <origin xyz="0.0421 0 0.3" rpy="0 0 0"/>
-        <limit effort="20" velocity="2.0" lower="-1.57" upper="1.57"/>
         <axis xyz=" 1 0 0"/>
     </joint>
@@ -202,5 +198,4 @@
         <child link="gripper_claw_link"/>
         <origin xyz="0.005725 0 0.07" rpy="0 0 0"/>
-        <limit effort="20" velocity="2.0" lower="-3.14" upper="3.14"/>
         <axis xyz="0 0 1"/>
     </joint>
@@ -209,5 +204,4 @@
         <child link="right_claw_link"/>
         <origin xyz="0 0.036895 0.135" rpy="0 0 0"/>
-        <limit effort="20" velocity="2.0" lower="0" upper="0.0275"/>
         <axis xyz="0 1 0"/>
     </joint>
@@ -216,5 +210,4 @@
         <child link="left_claw_link"/>
         <origin xyz="0 -0.036895 0.135" rpy="0 0 0"/>
-        <limit effort="20" velocity="2.0" lower="-0.0275" upper="0"/>
         <axis xyz="0 1 0"/>
     </joint>
