Commit message: added 6dof

File: src/ceres_moveit_config/config/ceres_rover.ros2_control.xacro (robot description, xacro)
@@ -6,7 +6,5 @@
             <hardware>
                 <!-- By default, set up controllers for simulation. This won't work on real hardware -->
-                <plugin>arm_hardware/RobotSystem</plugin>
-                        <!-- library_name/ClassName -->
-                <param name="port">/dev/ttyUSB0</param>
+                <plugin>mock_components/GenericSystem</plugin>
             </hardware>
             <joint name="joint1">
@@ -31,4 +29,11 @@
                 <state_interface name="velocity"/>
             </joint>
+            <joint name="joint4">
+                <command_interface name="position"/>
+                <state_interface name="position">
+                  <param name="initial_value">${initial_positions['joint4']}</param>
+                </state_interface>
+                <state_interface name="velocity"/>
+            </joint>
             <joint name="joint5">
                 <command_interface name="position"/>

File: src/ceres_urdf/urdf/ceres.xacro (robot description, xacro)
@@ -150,5 +150,5 @@
         <axis xyz="1 0 0"/>
     </joint>
-   <joint name="joint4" type="fixed">
+   <joint name="joint4" type="continuous">
         <parent link="bicep_gearbox_link"/>
         <child link="forearm_tube_link"/>

Commit message: modified moveit_config to implement gripper

File: src/ceres_moveit_config/config/ceres_rover.ros2_control.xacro (robot description, xacro)
@@ -50,4 +50,18 @@
                 <state_interface name="velocity"/>
             </joint>
+            <joint name="joint8">
+                <command_interface name="position"/>
+                <state_interface name="position">
+                  <param name="initial_value">${initial_positions['joint8']}</param>
+                </state_interface>
+                <state_interface name="velocity"/>
+            </joint>
+            <joint name="joint9">
+                <command_interface name="position"/>
+                <state_interface name="position">
+                  <param name="initial_value">${initial_positions['joint9']}</param>
+                </state_interface>
+                <state_interface name="velocity"/>
+            </joint>
         </ros2_control>
     </xacro:macro>

Commit message: set moveit_config for 5dof for proper hardware_interface test

File: src/ceres_moveit_config/config/ceres_rover.ros2_control.xacro (robot description, xacro)
@@ -29,11 +29,4 @@
                 <state_interface name="velocity"/>
             </joint>
-            <joint name="joint4">
-                <command_interface name="position"/>
-                <state_interface name="position">
-                  <param name="initial_value">${initial_positions['joint4']}</param>
-                </state_interface>
-                <state_interface name="velocity"/>
-            </joint>
             <joint name="joint5">
                 <command_interface name="position"/>
@@ -43,25 +36,4 @@
                 <state_interface name="velocity"/>
             </joint>
-            <joint name="joint7">
-                <command_interface name="position"/>
-                <state_interface name="position">
-                  <param name="initial_value">${initial_positions['joint7']}</param>
-                </state_interface>
-                <state_interface name="velocity"/>
-            </joint>
-            <joint name="joint8">
-                <command_interface name="position"/>
-                <state_interface name="position">
-                  <param name="initial_value">${initial_positions['joint8']}</param>
-                </state_interface>
-                <state_interface name="velocity"/>
-            </joint>
-            <joint name="joint9">
-                <command_interface name="position"/>
-                <state_interface name="position">
-                  <param name="initial_value">${initial_positions['joint9']}</param>
-                </state_interface>
-                <state_interface name="velocity"/>
-            </joint>
         </ros2_control>
     </xacro:macro>

File: src/ceres_urdf/urdf/ceres.xacro (robot description, xacro)
@@ -180,5 +180,5 @@
         <axis xyz="1 0 0"/>
     </joint>
-   <joint name="joint4" type="continuous">
+   <joint name="joint4" type="fixed">
         <parent link="bicep_gearbox_link"/>
         <child link="forearm_tube_link"/>
@@ -198,5 +198,5 @@
         <origin xyz="-0.026225 0 0.070075" rpy="0 0 0"/>
     </joint>
-    <joint name="joint7" type="revolute">
+    <joint name="joint7" type="fixed">
         <parent link="wrist_gearbox_link"/>
         <child link="gripper_claw_link"/>
@@ -205,5 +205,5 @@
         <axis xyz="0 0 1"/>
     </joint>
-    <joint name="joint8" type="prismatic">
+    <joint name="joint8" type="fixed">
         <parent link="gripper_claw_link"/>
         <child link="right_claw_link"/>
@@ -212,5 +212,5 @@
         <axis xyz="0 1 0"/>
     </joint>
-    <joint name="joint9" type="prismatic">
+    <joint name="joint9" type="fixed">
         <parent link="gripper_claw_link"/>
         <child link="left_claw_link"/>

Commit message: modified moveit_config for ik testing on arm

File: src/ceres_moveit_config/config/ceres_rover.ros2_control.xacro (robot description, xacro)
@@ -10,4 +10,5 @@
             <joint name="joint1">
                 <command_interface name="position"/>
+                <command_interface name="velocity"/>
                 <state_interface name="position">
                   <param name="initial_value">${initial_positions['joint1']}</param>
@@ -17,4 +18,5 @@
             <joint name="joint2">
                 <command_interface name="position"/>
+                <command_interface name="velocity"/>
                 <state_interface name="position">
                   <param name="initial_value">${initial_positions['joint2']}</param>
@@ -24,4 +26,5 @@
             <joint name="joint3">
                 <command_interface name="position"/>
+                <command_interface name="velocity"/>
                 <state_interface name="position">
                   <param name="initial_value">${initial_positions['joint3']}</param>
@@ -31,6 +34,15 @@
             <joint name="joint5">
                 <command_interface name="position"/>
+                <command_interface name="velocity"/>
                 <state_interface name="position">
                   <param name="initial_value">${initial_positions['joint5']}</param>
+                </state_interface>
+                <state_interface name="velocity"/>
+            </joint>
+            <joint name="joint7">
+                <command_interface name="position"/>
+                <command_interface name="velocity"/>
+                <state_interface name="position">
+                  <param name="initial_value">${initial_positions['joint7']}</param>
                 </state_interface>
                 <state_interface name="velocity"/>

File: src/ceres_urdf/urdf/ceres.xacro (robot description, xacro)
@@ -198,5 +198,5 @@
         <origin xyz="-0.026225 0 0.070075" rpy="0 0 0"/>
     </joint>
-    <joint name="joint7" type="fixed">
+    <joint name="joint7" type="revolute">
         <parent link="wrist_gearbox_link"/>
         <child link="gripper_claw_link"/>

Commit message: solving hardware issues

File: src/ceres_moveit_config/config/ceres_rover.ros2_control.xacro (robot description, xacro)
@@ -37,11 +37,4 @@
                 <state_interface name="velocity"/>
             </joint>
-            <joint name="joint7">
-                <command_interface name="position"/>
-                <state_interface name="position">
-                  <param name="initial_value">${initial_positions['joint7']}</param>
-                </state_interface>
-                <state_interface name="velocity"/>
-            </joint>
         </ros2_control>
     </xacro:macro>

Commit message: changes

File: src/ceres_moveit_config/config/ceres_rover.ros2_control.xacro (robot description, xacro)
@@ -5,10 +5,10 @@
         <ros2_control name="${name}" type="system">
             <hardware>
-                <!-- Use the actual hardware interface for the arm -->
+                <!-- By default, set up controllers for simulation. This won't work on real hardware -->
                 <plugin>arm_interface/ArmInterface</plugin>
-                <param name="port_name">/dev/ttyTHS1</param>
             </hardware>
             <joint name="joint1">
                 <command_interface name="position"/>
+                <command_interface name="velocity"/>
                 <state_interface name="position">
                   <param name="initial_value">${initial_positions['joint1']}</param>
@@ -18,4 +18,5 @@
             <joint name="joint2">
                 <command_interface name="position"/>
+                <command_interface name="velocity"/>
                 <state_interface name="position">
                   <param name="initial_value">${initial_positions['joint2']}</param>
@@ -25,4 +26,5 @@
             <joint name="joint3">
                 <command_interface name="position"/>
+                <command_interface name="velocity"/>
                 <state_interface name="position">
                   <param name="initial_value">${initial_positions['joint3']}</param>
@@ -32,6 +34,15 @@
             <joint name="joint5">
                 <command_interface name="position"/>
+                <command_interface name="velocity"/>
                 <state_interface name="position">
                   <param name="initial_value">${initial_positions['joint5']}</param>
+                </state_interface>
+                <state_interface name="velocity"/>
+            </joint>
+            <joint name="joint7">
+                <command_interface name="position"/>
+                <command_interface name="velocity"/>
+                <state_interface name="position">
+                  <param name="initial_value">${initial_positions['joint7']}</param>
                 </state_interface>
                 <state_interface name="velocity"/>

Commit message: modified ik files

File: src/ceres_moveit_config/config/ceres_rover.ros2_control.xacro (robot description, xacro)
@@ -10,5 +10,4 @@
             <joint name="joint1">
                 <command_interface name="position"/>
-                <command_interface name="velocity"/>
                 <state_interface name="position">
                   <param name="initial_value">${initial_positions['joint1']}</param>
@@ -18,5 +17,4 @@
             <joint name="joint2">
                 <command_interface name="position"/>
-                <command_interface name="velocity"/>
                 <state_interface name="position">
                   <param name="initial_value">${initial_positions['joint2']}</param>
@@ -26,5 +24,4 @@
             <joint name="joint3">
                 <command_interface name="position"/>
-                <command_interface name="velocity"/>
                 <state_interface name="position">
                   <param name="initial_value">${initial_positions['joint3']}</param>
@@ -34,15 +31,6 @@
             <joint name="joint5">
                 <command_interface name="position"/>
-                <command_interface name="velocity"/>
                 <state_interface name="position">
                   <param name="initial_value">${initial_positions['joint5']}</param>
-                </state_interface>
-                <state_interface name="velocity"/>
-            </joint>
-            <joint name="joint7">
-                <command_interface name="position"/>
-                <command_interface name="velocity"/>
-                <state_interface name="position">
-                  <param name="initial_value">${initial_positions['joint7']}</param>
                 </state_interface>
                 <state_interface name="velocity"/>

File: src/ceres_urdf/urdf/ceres.xacro (robot description, xacro)
@@ -198,5 +198,5 @@
         <origin xyz="-0.026225 0 0.070075" rpy="0 0 0"/>
     </joint>
-    <joint name="joint7" type="revolute">
+    <joint name="joint7" type="fixed">
         <parent link="wrist_gearbox_link"/>
         <child link="gripper_claw_link"/>

Commit message: fix bug

File: src/ceres_moveit_config/config/ceres_rover.ros2_control.xacro (robot description, xacro)
@@ -2,5 +2,5 @@
 <robot xmlns:xacro="http://www.ros.org/wiki/xacro">
     <xacro:macro name="ceres_rover_ros2_control" params="name initial_positions_file">
-        <xacro:property name="initial_positions" value="${load_yaml(initial_positions_file)['initial_positions']}"/>
+        <xacro:property name="initial_positions" value="${xacro.load_yaml(initial_positions_file)['initial_positions']}"/>
         <ros2_control name="${name}" type="system">
             <hardware>

Commit message: debugging launch files

File: src/ceres_moveit_config/config/ceres_rover.ros2_control.xacro (robot description, xacro)
@@ -5,5 +5,5 @@
         <ros2_control name="${name}" type="system">
             <hardware>
-                <!-- By default, set up controllers for simulation. This won't work on real hardware -->
+                <!-- By default, set up controllers for simulation. This won't work on real hardware (arm_interface/ArmInterface)-->
                 <plugin>arm_interface/ArmInterface</plugin>
             </hardware>

File: src/ceres_urdf/urdf/ceres.xacro (robot description, xacro)
@@ -1,3 +1,3 @@
-<?xml version="2.0"?>
+<?xml version="1.0"?>
 <robot name="ceres_rover" xmlns:xacro="http://www.ros.org/wiki/xacro">
     <material name="blue" >
@@ -183,5 +183,5 @@
         <axis xyz=" 0 0 1"/>
     </joint>
-    <joint name="joint5" type="revolute">
+    <joint name="joint5" type="continuous">
         <parent link="forearm_tube_link"/>
         <child link="bracket_connection_link"/>
