Commit message: pose typing

File: src/install/ceres_moveit_config/share/ceres_moveit_config/config/ceres_rover.ros2_control.xacro (robot description, xacro)
@@ -29,11 +29,4 @@
                 <state_interface name="velocity"/>
             </joint>
-            <joint name="joint4">
-                <command_interface name="position"/>
-                <state_interface name="position">
-                  <param name="initial_value">${initial_positions['joint4']}</param>
-                </state_interface>
-                <state_interface name="velocity"/>
-            </joint>
             <joint name="joint5">
                 <command_interface name="position"/>
@@ -43,11 +36,4 @@
                 <state_interface name="velocity"/>
             </joint>
-            <joint name="joint7">
-                <command_interface name="position"/>
-                <state_interface name="position">
-                  <param name="initial_value">${initial_positions['joint7']}</param>
-                </state_interface>
-                <state_interface name="velocity"/>
-            </joint>
         </ros2_control>
     </xacro:macro>
