Commit message: merge

File: src/inverse-kinematics/install/rover_arm_moveit_config/share/rover_arm_moveit_config/config/rover_arm.ros2_control.xacro (robot description, xacro)
@@ -8,8 +8,12 @@
                 <plugin>mock_components/GenericSystem</plugin>
             </hardware>
+<<<<<<< HEAD:src/ceres_moveit_config/config/ceres_rover.ros2_control.xacro
+            <joint name="joint1">
+=======
             <!-- Note: RVIZ only takes positional command interfaces, so when using this interface on the real arm
               one can simply comment out or remove the position command interfaces.-->
             <joint name="joint1">
                 <command_interface name="velocity"/>
+>>>>>>> main:src/inverse-kinematics/rover_arm_moveit_config/config/rover_arm.ros2_control.xacro
                 <command_interface name="position"/>
                 <state_interface name="position">
@@ -19,5 +23,8 @@
             </joint>
             <joint name="joint2">
+<<<<<<< HEAD:src/ceres_moveit_config/config/ceres_rover.ros2_control.xacro
+=======
                 <command_interface name="velocity"/>
+>>>>>>> main:src/inverse-kinematics/rover_arm_moveit_config/config/rover_arm.ros2_control.xacro
                 <command_interface name="position"/>
                 <state_interface name="position">
@@ -27,5 +34,8 @@
             </joint>
             <joint name="joint3">
+<<<<<<< HEAD:src/ceres_moveit_config/config/ceres_rover.ros2_control.xacro
+=======
                 <command_interface name="velocity"/>
+>>>>>>> main:src/inverse-kinematics/rover_arm_moveit_config/config/rover_arm.ros2_control.xacro
                 <command_interface name="position"/>
                 <state_interface name="position">
@@ -35,5 +45,8 @@
             </joint>
             <joint name="joint5">
+<<<<<<< HEAD:src/ceres_moveit_config/config/ceres_rover.ros2_control.xacro
+=======
                 <command_interface name="velocity"/>
+>>>>>>> main:src/inverse-kinematics/rover_arm_moveit_config/config/rover_arm.ros2_control.xacro
                 <command_interface name="position"/>
                 <state_interface name="position">
