Commit message: removed right_finger from moooveit_configs

File: src/inverse-kinematics/rover_arm_description/urdf/gripper.xacro (robot description, xacro)
@@ -46,5 +46,5 @@
         </collision>
     </link>
-    <joint name="right_finger" type="prismatic">
+    <joint name="right_finger" type="fixed">
         <parent link="gripper_claw_link"/>
         <child link="right_claw_link"/>
@@ -53,5 +53,5 @@
         <limit lower="0.0" upper="0.033" effort="100.0" velocity="1.0"/>
     </joint>
-    <joint name="left_finger" type="prismatic">
+    <joint name="left_finger" type="fixed">
         <parent link="gripper_claw_link"/>
         <child link="left_claw_link"/>

Commit message: added servo control?

File: src/inverse-kinematics/rover_arm_description/urdf/gripper.xacro (robot description, xacro)
@@ -46,5 +46,5 @@
         </collision>
     </link>
-    <joint name="right_finger" type="fixed">
+    <joint name="right_finger" type="prismatic">
         <parent link="gripper_claw_link"/>
         <child link="right_claw_link"/>
@@ -53,5 +53,5 @@
         <limit lower="0.0" upper="0.033" effort="100.0" velocity="1.0"/>
     </joint>
-    <joint name="left_finger" type="fixed">
+    <joint name="left_finger" type="prismatic">
         <parent link="gripper_claw_link"/>
         <child link="left_claw_link"/>
