Commit message: changed ar lengths

File: src/inverse-kinematics/rover_arm_description/urdf/arm.xacro (robot description, xacro)
@@ -34,5 +34,5 @@
         <visual>
             <geometry>
-                <cylinder radius="0.0348" length="0.520"/>
+                <cylinder radius="0.0348" length="0.508"/>
             </geometry>
             <origin xyz="0 0 0.220" rpy="0 0 0"/>
@@ -41,5 +41,5 @@
         <collision>
             <geometry>
-                <cylinder radius="0.0348" length="0.520"/>
+                <cylinder radius="0.0348" length="0.508"/>
             </geometry>
             <material name="grey"/>
@@ -64,5 +64,5 @@
         <visual>
             <geometry>
-                <cylinder radius="0.03810" length="0.300"/>
+                <cylinder radius="0.03810" length="0.490"/>
             </geometry>
             <origin xyz="0 0 0.150" rpy="0 0 0"/>
@@ -71,5 +71,5 @@
         <collision>
             <geometry>
-                <cylinder radius="0.03810" length="0.300"/>
+                <cylinder radius="0.03810" length="0.490"/>
             </geometry>
             <material name="grey"/>

Commit message: Added axis of rotation to joint 3

File: src/inverse-kinematics/rover_arm_description/urdf/arm.xacro (robot description, xacro)
@@ -116,4 +116,5 @@
         <child link="bicep_tube_link"/>
         <origin xyz="0.11645 0 0" rpy="0 0 0"/>
+        <axis xyz="1 0 0"/>
     </joint>
     <joint name="joint3" type="continuous">

Commit message: Fixed orientation of tf's in URDF

File: src/inverse-kinematics/rover_arm_description/urdf/arm.xacro (robot description, xacro)
@@ -6,5 +6,5 @@
                 <box size="0.30670 0.1600 0.135"/>
             </geometry>
-            <origin xyz="0 0 0" rpy="1.57 0 0" />
+            <origin xyz="0 0 0" rpy="0 0 1.57" />
             <material name="blue"/>
         </visual>
@@ -51,5 +51,5 @@
                 <box size="0.11615 0.158 0.170"/>
             </geometry>
-            <origin xyz="0 0 0" rpy="0 0 0"/>
+            <origin xyz="0 0 0" rpy="0 0 1.57"/>
             <material name="red"/>
         </visual>
@@ -81,10 +81,10 @@
                 <box size="0.008 0.10030 0.14015"/>
             </geometry>
-            <origin xyz="0 0 0" rpy="0 0 0"/>
+            <origin xyz="0 0 0" rpy="0 0 -1.57"/>
             <material name="grey"/>
         </visual>
         <collision>
             <geometry>
-                <box size="0 0 0"/>
+                <box size="0.008 0.10030 0.14015"/>
             </geometry>
             <material name="grey"/>
@@ -96,10 +96,10 @@
                 <box size="0.04445 0.06200 0.07"/>
             </geometry>
-            <origin xyz="0 0 0" rpy="0 0 0"/>
+            <origin xyz="0 0 0" rpy="0 0 -1.57"/>
             <material name="grey"/>
         </visual>
         <collision>
             <geometry>
-                <box size="0 0 0"/>
+                <box size="0.04445 0.06200 0.07"/>
             </geometry>
             <material name="grey"/>
@@ -115,12 +115,12 @@
         <parent link="base_pivot_link"/>
         <child link="bicep_tube_link"/>
-        <origin xyz="0.11645 0 0" rpy="0 0 0"/>
-        <axis xyz="1 0 0"/>
+        <origin xyz="0 0.11645 0" rpy="0 0 0"/>
+        <axis xyz="0 1 0"/>
     </joint>
     <joint name="joint3" type="continuous">
         <parent link="bicep_tube_link"/>
         <child link="bicep_gearbox_link"/>
-        <origin xyz="-0.092875 0 0.440" rpy="0 0 0"/>
-        <axis xyz="1 0 0"/>
+        <origin xyz="0 -0.092875 0.440" rpy="0 0 0"/>
+        <axis xyz="0 1 0"/>
     </joint>
    <joint name="joint4" type="fixed">
@@ -133,11 +133,11 @@
         <parent link="forearm_tube_link"/>
         <child link="bracket_connection_link"/>
-        <origin xyz="0.0421 0 0.3" rpy="0 0 0"/>
-        <axis xyz=" 1 0 0"/>
+        <origin xyz="0 -0.0421 0.35" rpy="0 0 0"/>
+        <axis xyz=" 0 1 0"/>
     </joint>
     <joint name="joint6" type="fixed">
         <parent link="bracket_connection_link"/>
         <child link="gripper_base_link"/>
-        <origin xyz="-0.026225 0 0.070075" rpy="0 0 0"/>
+        <origin xyz="0 0 0.085075" rpy="0 0 0"/>
     </joint>
 </robot>

File: src/inverse-kinematics/rover_arm_description/urdf/gripper.xacro (robot description, xacro)
@@ -6,5 +6,5 @@
                 <box size="0.033 0.14759 0.070"/>
             </geometry>
-            <origin xyz="0 0 0" rpy="0 0 0"/>
+            <origin xyz="0 0 0" rpy="0 0 -1.57"/>
             <material name="blue"/>
         </visual>
@@ -21,5 +21,5 @@
                 <box size="0.033 0.073795 0.200"/>
             </geometry>
-            <origin xyz="0 0 0" rpy="0 0 0"/>
+            <origin xyz="0 0 0" rpy="0 0 1.57"/>
             <material name="red"/>
         </visual>
@@ -36,5 +36,5 @@
                 <box size="0.033 0.073795 0.200"/>
             </geometry>
-            <origin xyz="0 0 0" rpy="0 0 0"/>
+            <origin xyz="0 0 0" rpy="0 0 1.57"/>
             <material name="red"/>
         </visual>
@@ -49,5 +49,5 @@
         <parent link="gripper_claw_link"/>
         <child link="right_claw_link"/>
-        <origin xyz="0 0.036895 0.135" rpy="0 0 0"/>
+        <origin xyz="0.036895 0 0.135" rpy="0 0 0"/>
         <axis xyz="0 1 0"/>
         <limit lower="0.0" upper="0.033" effort="100.0" velocity="1.0"/>
@@ -56,5 +56,5 @@
         <parent link="gripper_claw_link"/>
         <child link="left_claw_link"/>
-        <origin xyz="0 -0.036895 0.135" rpy="0 0 0"/>
+        <origin xyz="-0.036895 0 0.135" rpy="0 0 0"/>
         <axis xyz="0 1 0"/>
         <mimic joint="right_finger" multiplier="-1.0"/>

Commit message: added joint limits

File: src/inverse-kinematics/rover_arm_description/urdf/arm.xacro (robot description, xacro)
@@ -106,21 +106,24 @@
         </collision>
     </link>
-    <joint name="joint1" type="continuous">
+    <joint name="joint1" type="revolute">
         <parent link="base_structure_link"/>
         <child link="base_pivot_link"/>
         <origin xyz="0 0 0.1618" rpy="0 0 0"/>
         <axis xyz="0 0 1"/>
+        <limit effort="100.0" lower="-1.57" upper="1.57" velocity="1.0" />
     </joint>
-    <joint name="joint2" type="continuous">
+    <joint name="joint2" type="revolute">
         <parent link="base_pivot_link"/>
         <child link="bicep_tube_link"/>
         <origin xyz="0 0.11645 0" rpy="0 0 0"/>
         <axis xyz="0 1 0"/>
+        <limit effort="100.0" lower="-0.701" upper="1.09" velocity="1.0" />
     </joint>
-    <joint name="joint3" type="continuous">
+    <joint name="joint3" type="revolute">
         <parent link="bicep_tube_link"/>
         <child link="bicep_gearbox_link"/>
         <origin xyz="0 -0.092875 0.440" rpy="0 0 0"/>
         <axis xyz="0 1 0"/>
+        <limit effort="100.0" lower="0.0" upper="2.109" velocity="1.0" />
     </joint>
    <joint name="joint4" type="fixed">
@@ -130,9 +133,10 @@
         <axis xyz=" 0 0 1"/>
     </joint>
-    <joint name="joint5" type="continuous">
+    <joint name="joint5" type="revolute">
         <parent link="forearm_tube_link"/>
         <child link="bracket_connection_link"/>
         <origin xyz="0 -0.0421 0.35" rpy="0 0 0"/>
         <axis xyz=" 0 1 0"/>
+        <limit effort="100.0" lower="-1.09" upper="1.57" velocity="1.0" />
     </joint>
     <joint name="joint6" type="fixed">
