Commit message: modified new rover_arm_description

File: src/inverse-kinematics/rover_arm_description/urdf/arm.urdf.xacro (robot description, xacro)
@@ -4,8 +4,9 @@
     <xacro:include filename="gripper.xacro"/>
     <xacro:include filename="common_properties.xacro"/>
-    <joint name="gripper_base_joint" type="fixed">
-        <parent link="bracket_connection_link"/>
-        <child link="gripper_base_link"/>
-        <origin xyz="-0.026225 0 0.070075" rpy="0 0 0"/>
+    <joint name="joint7" type="fixed">
+        <parent link="gripper_base_link"/>
+        <child link="gripper_claw_link"/>
+        <origin xyz="0.005725 0 0.07" rpy="0 0 0"/>
+        <axis xyz="0 0 1"/>
     </joint>
 </robot>

File: src/inverse-kinematics/rover_arm_description/urdf/arm.xacro (robot description, xacro)
@@ -91,4 +91,19 @@
         </collision>
     </link>
+    <link name="gripper_base_link">
+        <visual>
+            <geometry>
+                <box size="0.04445 0.06200 0.07"/>
+            </geometry>
+            <origin xyz="0 0 0" rpy="0 0 0"/>
+            <material name="grey"/>
+        </visual>
+        <collision>
+            <geometry>
+                <box size="0 0 0"/>
+            </geometry>
+            <material name="grey"/>
+        </collision>
+    </link>
     <joint name="joint1" type="continuous">
         <parent link="base_structure_link"/>
@@ -120,3 +135,8 @@
         <axis xyz=" 1 0 0"/>
     </joint>
+    <joint name="joint6" type="fixed">
+        <parent link="bracket_connection_link"/>
+        <child link="gripper_base_link"/>
+        <origin xyz="-0.026225 0 0.070075" rpy="0 0 0"/>
+    </joint>
 </robot>

File: src/inverse-kinematics/rover_arm_description/urdf/gripper.xacro (robot description, xacro)
@@ -1,19 +1,4 @@
 <?xml version="1.0"?>
 <robot xmlns:xacro="http://www.ros.org/wiki/xacro">
-    <link name="gripper_base_link">
-        <visual>
-            <geometry>
-                <box size="0.04445 0.06200 0.07"/>
-            </geometry>
-            <origin xyz="0 0 0" rpy="0 0 0"/>
-            <material name="grey"/>
-        </visual>
-        <collision>
-            <geometry>
-                <box size="0 0 0"/>
-            </geometry>
-            <material name="grey"/>
-        </collision>
-    </link>
     <link name="gripper_claw_link">
         <visual>
@@ -61,10 +46,4 @@
         </collision>
     </link>
-    <joint name="joint7" type="fixed">
-        <parent link="gripper_base_link"/>
-        <child link="gripper_claw_link"/>
-        <origin xyz="0.005725 0 0.07" rpy="0 0 0"/>
-        <axis xyz="0 0 1"/>
-    </joint>
     <joint name="right_finger" type="fixed">
         <parent link="gripper_claw_link"/>

Commit message: implemented gripper and servo rotation to Ik

File: src/inverse-kinematics/rover_arm_description/urdf/arm.urdf.xacro (robot description, xacro)
@@ -5,5 +5,5 @@
     <xacro:include filename="common_properties.xacro"/>
     <!-- <xacro:include filename="rover_arm.ros2_control.xacro"/> -->
-    <joint name="joint7" type="fixed">
+    <joint name="joint7" type="continuous">
         <parent link="gripper_base_link"/>
         <child link="gripper_claw_link"/>

File: src/inverse-kinematics/rover_arm_description/urdf/gripper.xacro (robot description, xacro)
@@ -46,15 +46,18 @@
         </collision>
     </link>
-    <joint name="right_finger" type="fixed">
+    <joint name="right_finger" type="prismatic">
         <parent link="gripper_claw_link"/>
         <child link="right_claw_link"/>
         <origin xyz="0 0.036895 0.135" rpy="0 0 0"/>
         <axis xyz="0 1 0"/>
+        <limit lower="0.0" upper="0.033" effort="100.0" velocity="1.0"/>
     </joint>
-    <joint name="left_finger" type="fixed">
+    <joint name="left_finger" type="prismatic">
         <parent link="gripper_claw_link"/>
         <child link="left_claw_link"/>
         <origin xyz="0 -0.036895 0.135" rpy="0 0 0"/>
         <axis xyz="0 1 0"/>
+        <mimic joint="right_finger" multiplier="-1.0"/>
+        <limit lower="-0.033" upper="0.0" effort="100.0" velocity="1.0"/>
     </joint>
 </robot>

File: src/inverse-kinematics/rover_arm_moveit_config/config/rover_arm.ros2_control.xacro (robot description, xacro)
@@ -41,4 +41,20 @@
                 <state_interface name="velocity"/>
             </joint>
+            <joint name="joint7">
+                <command_interface name="velocity"/>
+                <!-- <command_interface name="position"/> -->
+                <state_interface name="position">
+                  <param name="initial_value">${initial_positions['joint7']}</param>
+                </state_interface>
+                <state_interface name="velocity"/>
+            </joint>
+            <joint name="right_finger">
+                <command_interface name="velocity"/>
+                <!-- <command_interface name="position"/> -->
+                <state_interface name="position">
+                  <param name="initial_value">${initial_positions['right_finger']}</param>
+                </state_interface>
+                <state_interface name="velocity"/>
+            </joint>
         </ros2_control>
     </xacro:macro>

Commit message: remove joint 7 from IK

File: src/inverse-kinematics/rover_arm_description/urdf/arm.urdf.xacro (robot description, xacro)
@@ -5,5 +5,5 @@
     <xacro:include filename="common_properties.xacro"/>
     <!-- <xacro:include filename="rover_arm.ros2_control.xacro"/> -->
-    <joint name="joint7" type="continuous">
+    <joint name="joint7" type="fixed">
         <parent link="gripper_base_link"/>
         <child link="gripper_claw_link"/>

File: src/inverse-kinematics/rover_arm_moveit_config/config/rover_arm.ros2_control.xacro (robot description, xacro)
@@ -41,5 +41,5 @@
                 <state_interface name="velocity"/>
             </joint>
-            <joint name="joint7">
+            <!-- <joint name="joint7">
                 <command_interface name="velocity"/>
                 <!-- <command_interface name="position"/> -->
@@ -48,5 +48,5 @@
                 </state_interface>
                 <state_interface name="velocity"/>
-            </joint>
+            </joint> -->
         </ros2_control>
     </xacro:macro>

Commit message: added 6 dof to urdf

File: src/inverse-kinematics/rover_arm_description/urdf/arm.urdf.xacro (robot description, xacro)
@@ -5,9 +5,10 @@
     <xacro:include filename="common_properties.xacro"/>
     <!-- <xacro:include filename="rover_arm.ros2_control.xacro"/> -->
-    <joint name="joint7" type="fixed">
+    <joint name="joint7" type="revolute">
         <parent link="gripper_base_link"/>
         <child link="gripper_claw_link"/>
         <origin xyz="0.005725 0 0.07" rpy="0 0 0"/>
         <axis xyz="0 0 1"/>
+        <limit effort="100.0" lower="-1.57" upper="1.57" velocity="1.0" />
     </joint>
 </robot>

File: src/inverse-kinematics/rover_arm_description/urdf/arm.xacro (robot description, xacro)
@@ -127,9 +127,10 @@
         <limit effort="100.0" lower="0.0" upper="2.109" velocity="1.0" />
     </joint>
-   <joint name="joint4" type="fixed">
+   <joint name="joint4" type="revolute">
         <parent link="bicep_gearbox_link"/>
         <child link="forearm_tube_link"/>
         <origin xyz="0 0 0.085" rpy="0 0 0"/>
         <axis xyz=" 0 0 1"/>
+        <limit effort="100.0" lower="-3.14159" upper="3.14159" velocity="1.0" />
     </joint>
     <joint name="joint5" type="revolute">
@@ -137,5 +138,5 @@
         <child link="bracket_connection_link"/>
         <origin xyz="0 -0.0421 0.35" rpy="0 0 0"/>
-        <axis xyz=" 0 1 0"/>
+        <axis xyz="0 1 0"/>
         <limit effort="100.0" lower="-1.09" upper="1.57" velocity="1.0" />
     </joint>

File: src/inverse-kinematics/rover_arm_moveit_config/config/rover_arm.ros2_control.xacro (robot description, xacro)
@@ -1,9 +1,14 @@
 <?xml version="1.0"?>
 <robot xmlns:xacro="http://www.ros.org/wiki/xacro">
-    <xacro:macro name="rover_arm_ros2_control" params="name initial_positions_file">
+    <xacro:macro name="rover_arm_ros2_control" params="name initial_positions_file use_fake_hardware:=false">
         <xacro:property name="initial_positions" value="${load_yaml(initial_positions_file)['initial_positions']}"/>
        <ros2_control name="RoverArm" type="system">
           <hardware>
-            <plugin>arm_interface/ArmInterface</plugin>
+            <xacro:if value="${use_fake_hardware}">
+              <plugin>mock_components/GenericSystem</plugin>
+            </xacro:if>
+            <xacro:unless value="${use_fake_hardware}">
+              <plugin>arm_interface/ArmInterface</plugin>
+            </xacro:unless>
             <param name="calculate_dynamics">true</param>
           </hardware>
@@ -31,4 +36,11 @@
                 <state_interface name="velocity"/>
             </joint>
+            <joint name="joint4">
+                <command_interface name="velocity"/>
+                <state_interface name="position">
+                  <param name="initial_value">${initial_positions['joint4']}</param>
+                </state_interface>
+                <state_interface name="velocity"/>
+            </joint>
             <joint name="joint5">
                 <command_interface name="velocity"/>
@@ -38,4 +50,11 @@
                 <state_interface name="velocity"/>
             </joint>
+            <joint name="joint7">
+                <command_interface name="velocity"/>
+                <state_interface name="position">
+                  <param name="initial_value">${initial_positions['joint7']}</param>
+                </state_interface>
+                <state_interface name="velocity"/>
+            </joint>
         </ros2_control>
     </xacro:macro>

File: src/inverse-kinematics/rover_arm_moveit_config/config/rover_arm.urdf.xacro (robot description, xacro)
@@ -2,8 +2,12 @@
 <robot xmlns:xacro="http://www.ros.org/wiki/xacro" name="rover_arm">
     <xacro:arg name="initial_positions_file" default="initial_positions.yaml" />
+    <xacro:arg name="use_fake_hardware" default="false" />
     <!-- Import rover_arm urdf file -->
     <xacro:include filename="$(find rover_arm_description)/urdf/arm.urdf.xacro" />
     <!-- Import control_xacro -->
     <xacro:include filename="rover_arm.ros2_control.xacro" />
-    <xacro:rover_arm_ros2_control name="FakeSystem" initial_positions_file="$(arg initial_positions_file)"/>
+        <xacro:rover_arm_ros2_control
+            name="FakeSystem"
+            initial_positions_file="$(arg initial_positions_file)"
+            use_fake_hardware="$(arg use_fake_hardware)"/>
 </robot>
