Commit message: removed gripper from servo

File: src/inverse-kinematics/rover_arm_moveit_config/config/rover_arm.ros2_control.xacro (robot description, xacro)
@@ -49,5 +49,5 @@
                 <state_interface name="velocity"/>
             </joint>
-            <joint name="right_finger">
+            <!-- <joint name="right_finger">
                 <command_interface name="velocity"/>
                 <!-- <command_interface name="position"/> -->
@@ -56,5 +56,5 @@
                 </state_interface>
                 <state_interface name="velocity"/>
-            </joint>
+            </joint> -->
         </ros2_control>
     </xacro:macro>

Commit message: removed right finger instances

File: src/inverse-kinematics/rover_arm_moveit_config/config/rover_arm.ros2_control.xacro (robot description, xacro)
@@ -49,12 +49,4 @@
                 <state_interface name="velocity"/>
             </joint>
-            <!-- <joint name="right_finger">
-                <command_interface name="velocity"/>
-                 <command_interface name="position"/>
-                <state_interface name="position">
-                  <param name="initial_value">${initial_positions['right_finger']}</param>
-                </state_interface>
-                <state_interface name="velocity"/>
-            </joint> -->
         </ros2_control>
     </xacro:macro>

Commit message: more changes

File: src/inverse-kinematics/rover_arm_moveit_config/config/rover_arm.ros2_control.xacro (robot description, xacro)
@@ -41,12 +41,4 @@
                 <state_interface name="velocity"/>
             </joint>
-            <!-- <joint name="joint7">
-                <command_interface name="velocity"/>
-                <!-- <command_interface name="position"/> -->
-                <state_interface name="position">
-                  <param name="initial_value">${initial_positions['joint7']}</param>
-                </state_interface>
-                <state_interface name="velocity"/>
-            </joint> -->
         </ros2_control>
     </xacro:macro>

Commit message: fix?

File: src/inverse-kinematics/rover_arm_moveit_config/config/rover_arm.ros2_control.xacro (robot description, xacro)
@@ -9,12 +9,4 @@
             <!-- Note: RVIZ only takes positional command interfaces, so when using this interface on the real arm
               one can simply comment out or remove the position command interfaces.-->
-            <joint name="joint1">
-                <command_interface name="velocity"/>
-                <!-- <command_interface name="position"/> -->
-                <state_interface name="position">
-                  <param name="initial_value">${initial_positions['joint1']}</param>
-                </state_interface>
-                <state_interface name="velocity"/>
-            </joint>
             <joint name="joint2">
                 <command_interface name="velocity"/>
@@ -41,4 +33,12 @@
                 <state_interface name="velocity"/>
             </joint>
+            <joint name="joint1">
+                <command_interface name="velocity"/>
+                <!-- <command_interface name="position"/> -->
+                <state_interface name="position">
+                  <param name="initial_value">${initial_positions['joint1']}</param>
+                </state_interface>
+                <state_interface name="velocity"/>
+            </joint>
         </ros2_control>
     </xacro:macro>

Commit message: reverted changes

File: src/inverse-kinematics/rover_arm_moveit_config/config/rover_arm.ros2_control.xacro (robot description, xacro)
@@ -9,4 +9,12 @@
             <!-- Note: RVIZ only takes positional command interfaces, so when using this interface on the real arm
               one can simply comment out or remove the position command interfaces.-->
+            <joint name="joint1">
+                <command_interface name="velocity"/>
+                <!-- <command_interface name="position"/> -->
+                <state_interface name="position">
+                  <param name="initial_value">${initial_positions['joint1']}</param>
+                </state_interface>
+                <state_interface name="velocity"/>
+            </joint>
             <joint name="joint2">
                 <command_interface name="velocity"/>
@@ -33,12 +41,4 @@
                 <state_interface name="velocity"/>
             </joint>
-            <joint name="joint1">
-                <command_interface name="velocity"/>
-                <!-- <command_interface name="position"/> -->
-                <state_interface name="position">
-                  <param name="initial_value">${initial_positions['joint1']}</param>
-                </state_interface>
-                <state_interface name="velocity"/>
-            </joint>
         </ros2_control>
     </xacro:macro>

Commit message: added independed servos

File: src/inverse-kinematics/rover_arm_moveit_config/config/rover_arm.ros2_control.xacro (robot description, xacro)
@@ -1,7 +1,7 @@
 <?xml version="1.0"?>
 <robot xmlns:xacro="http://www.ros.org/wiki/xacro">
-    <xacro:macro name="rover_arm_ros2_control" params="name initial_positions_file">
+    <xacro:macro name="rover_servo_ros2_control" params="name initial_positions_file">
         <xacro:property name="initial_positions" value="${load_yaml(initial_positions_file)['initial_positions']}"/>
-       <ros2_control name="RoverArm" type="system">
+       <ros2_control name="RoverServo" type="system">
           <hardware>
             <plugin>arm_interface/ArmInterface</plugin>
@@ -41,20 +41,4 @@
                 <state_interface name="velocity"/>
             </joint>
-            <joint name="joint7">
-                <command_interface name="velocity"/>
-                <!-- <command_interface name="position"/> -->
-                <state_interface name="position">
-                  <param name="initial_value">${initial_positions['joint7']}</param>
-                </state_interface>
-                <state_interface name="velocity"/>
-            </joint>
-            <joint name="right_finger">
-                <command_interface name="velocity"/>
-                <!-- <command_interface name="position"/> -->
-                <state_interface name="position">
-                  <param name="initial_value">${initial_positions['right_finger']}</param>
-                </state_interface>
-                <state_interface name="velocity"/>
-            </joint>
         </ros2_control>
     </xacro:macro>

File: src/inverse-kinematics/rover_arm_moveit_config/config/rover_arm.urdf.xacro (robot description, xacro)
@@ -6,4 +6,6 @@
     <!-- Import control_xacro -->
     <xacro:include filename="rover_arm.ros2_control.xacro" />
-    <xacro:rover_arm_ros2_control name="FakeSystem" initial_positions_file="$(arg initial_positions_file)"/>
+    <xacro:include filename="arm_servo.ros2_control.xacro" />
+    <xacro:rover_arm_ros2_control name="RoverArm" initial_positions_file="$(arg initial_positions_file)"/>
+    <xacro:rover_servo_ros2_control name="RoverServo" initial_positions_file="$(arg initial_positions_file)"/>
 </robot>

Commit message: changed mappings, improved hardware interface, added a mapping checker, first part of encoder implementation

File: src/inverse-kinematics/rover_arm_moveit_config/config/rover_arm.ros2_control.xacro (robot description, xacro)
@@ -62,4 +62,19 @@
                 <state_interface name="velocity"/>
             </joint>
+            <!--
+              Gripper (CLAMP servo) via Firmware_SPIN MOVE_POSITION — see docs/SERVO_API.md.
+              Uncomment to enable ros2_control commanding of the gripper.
+              servo_max is max degrees per command tick (firmware clamps ±100°).
+            <joint name="joint7">
+                <param name="kind">clamp_servo</param>
+                <param name="servo_mode">move_position</param>
+                <param name="servo_max">15.0</param>
+                <command_interface name="velocity"/>
+                <state_interface name="position">
+                  <param name="initial_value">0.0</param>
+                </state_interface>
+                <state_interface name="velocity"/>
+            </joint>
+            -->
         </ros2_control>
     </xacro:macro>
