Commit message: Remove WIP ros2_control arm/wheel hardware from integration PR
Co-authored-by: Cursor <cursoragent@cursor.com>

File: src/inverse-kinematics/rover_arm_moveit_config/config/rover_arm.ros2_control.xacro (robot description, xacro)
@@ -5,22 +5,11 @@
        <ros2_control name="RoverArm" type="system">
           <hardware>
-            <!--
-              CAN-based hardware interface. The legacy serial plugin
-              (arm_interface/ArmInterface) is preserved in the arm_hardware
-              package for reference but is no longer wired here.
-            -->
-            <plugin>arm_can_hardware/ArmCanInterface</plugin>
-            <param name="can_interface">can0</param>
-            <param name="send_heartbeat_on_activate">true</param>
+            <plugin>arm_interface/ArmInterface</plugin>
           </hardware>
-            <!-- Per-joint parameters tell ArmCanInterface which CAN motor /
-                 encoder a URDF joint maps onto. arm_instruction values come
-                 from Instructions::Inst in can-utils/prefixes.hpp. -->
+            <!-- Note: RVIZ only takes positional command interfaces, so when using this interface on the real arm
+              one can simply comment out or remove the position command interfaces.-->
             <joint name="joint1">
-                <param name="kind">arm_motor</param>
-                <param name="arm_instruction">0x12</param>      <!-- ARM_MOTOR_1 -->
-                <param name="encoder_device_id">0x07</param>    <!-- BASE_ENCODER -->
-                <param name="velocity_scale">1.0</param>
                 <command_interface name="velocity"/>
+                <!-- <command_interface name="position"/> -->
                 <state_interface name="position">
                   <param name="initial_value">${initial_positions['joint1']}</param>
@@ -29,9 +18,6 @@
             </joint>
             <joint name="joint2">
-                <param name="kind">arm_motor</param>
-                <param name="arm_instruction">0x14</param>      <!-- ARM_MOTOR_2 -->
-                <param name="encoder_device_id">0x08</param>    <!-- SHOULDER_ENCODER -->
-                <param name="velocity_scale">1.0</param>
                 <command_interface name="velocity"/>
+                <!-- <command_interface name="position"/> -->
                 <state_interface name="position">
                   <param name="initial_value">${initial_positions['joint2']}</param>
@@ -40,10 +26,6 @@
             </joint>
             <joint name="joint3">
-                <param name="kind">arm_motor</param>
-                <param name="arm_instruction">0x16</param>      <!-- ARM_MOTOR_3 -->
-                <param name="encoder_device_id">0x09</param>    <!-- ELBOW_ENCODER -->
-                <param name="velocity_scale">1.0</param>
-                <param name="direction">-1.0</param>
                 <command_interface name="velocity"/>
+                <!-- <command_interface name="position"/> -->
                 <state_interface name="position">
                   <param name="initial_value">${initial_positions['joint3']}</param>
@@ -52,9 +34,6 @@
             </joint>
             <joint name="joint5">
-                <param name="kind">arm_motor</param>
-                <param name="arm_instruction">0x1A</param>      <!-- ARM_MOTOR_5 -->
-                <param name="encoder_device_id">0x0B</param>    <!-- WRIST_ENCODER -->
-                <param name="velocity_scale">1.0</param>
                 <command_interface name="velocity"/>
+                <!-- <command_interface name="position"/> -->
                 <state_interface name="position">
                   <param name="initial_value">${initial_positions['joint5']}</param>
@@ -62,19 +41,4 @@
                 <state_interface name="velocity"/>
             </joint>
-            <!--
-              Gripper (CLAMP servo) via Firmware_SPIN MOVE_POSITION — see docs/SERVO_API.md.
-              Uncomment to enable ros2_control commanding of the gripper.
-              servo_max is max degrees per command tick (firmware clamps ±100°).
-            <joint name="joint7">
-                <param name="kind">clamp_servo</param>
-                <param name="servo_mode">move_position</param>
-                <param name="servo_max">15.0</param>
-                <command_interface name="velocity"/>
-                <state_interface name="position">
-                  <param name="initial_value">0.0</param>
-                </state_interface>
-                <state_interface name="velocity"/>
-            </joint>
-            -->
         </ros2_control>
     </xacro:macro>
